Commit message: trying to figure out hand assembly

File: inmoov/inmoov_urdf/urdf/rightHand.urdf (robot description, URDF)
Before this commit: robot rightHand, 1 links, 0 joints
Links:
- added link wristPinky; visual mesh filename=package://inmoov/meshes/rightHand/wristSmallPinky.stl scale=.001 .001 .001
- added link wristRing; visual mesh filename=package://inmoov/meshes/rightHand/wristSmallRing.stl scale=.001 .001 .001
- link wristLarge: geometry visual mesh filename=package://inmoov/meshes/rightHand/WristlargeV4.stl scale=.001 .001 .001
Joints:
- added joint pinkyKnuck1: type revolute, parent wristLarge, child wristPinky, origin xyz=0 0 0, limit lower=0.0 upper=-0.35 effort=1000.0 velocity=-0.5
- added joint ringKnuck1: type revolute, parent wristLarge, child wristRing, origin xyz=0 -0.04 0, limit lower=0.0 upper=-0.35 effort=1000.0 velocity=-0.5

Commit message: almost have the wrist knuckles done and setup inmoov_urdf file structure to hopefully better work with ros indigo

File: inmoov/inmoov_urdf/urdf/rightHand.urdf (robot description, URDF)
Before this commit: robot rightHand, 3 links, 2 joints
Links:
- link wristLarge: geometry visual mesh filename=package://inmoov_urdf/meshes/rightHand/WristlargeV4.stl scale=.001 .001 .001
- link wristPinky: geometry visual mesh filename=package://inmoov_urdf/meshes/rightHand/wristSmallPinky.stl scale=.001 .001 .001
- link wristRing: geometry visual mesh filename=package://inmoov_urdf/meshes/rightHand/wristSmallRing.stl scale=.001 .001 .001
Joints:
- joint pinkyKnuck1: limit lower=0.0 upper=-0.35 effort=1000.0 velocity=-0.5 -> lower=0.0 upper=0.26 effort=1000.0 velocity=0.5; origin xyz=0 0 0 -> xyz=0.005 -0.0105 .0105 rpy=0 0 4.03171057
- joint ringKnuck1: limit lower=0.0 upper=-0.35 effort=1000.0 velocity=-0.5 -> lower=0.0 upper=0.26 effort=1000.0 velocity=0.5; origin xyz=0 -0.04 0 -> xyz=0.005 -0.0105 .0105 rpy=0 0 4.03171057

Commit message: fixed pinky and midlle wrist knuckle limits, added new mesh files for the index finger, and positioned the first index knuckle

File: inmoov/inmoov_urdf/urdf/rightHand.urdf (robot description, URDF)
Before this commit: robot rightHand, 3 links, 2 joints
Links:
- added link indexSeg6; visual mesh filename=package://inmoov_urdf/meshes/rightHand/indexSeg6.stl scale=.001 .001 .001
Joints:
- added joint indexKnuck1: type revolute, parent wristLarge, child indexSeg6, origin xyz=-0.0352 -0.0505 0.0107 rpy=0 0 -0.0875, limit lower=0.0 upper=-1.74533 effort=1000.0 velocity=0.5
- joint pinkyKnuck1: limit lower=0.0 upper=0.26 effort=1000.0 velocity=0.5 -> lower=0.0 upper=0.3 effort=1000.0 velocity=0.5
- joint ringKnuck1: limit lower=0.0 upper=0.26 effort=1000.0 velocity=0.5 -> lower=0.0 upper=0.23 effort=1000.0 velocity=0.5; origin xyz=0.005 -0.0105 .0105 rpy=0 0 4.03171057 -> xyz=0.005 -0.0105 0.0105 rpy=0 0 4.03171057

Commit message: finished modeling index finger joints

File: inmoov/inmoov_urdf/urdf/rightHand.urdf (robot description, URDF)
Before this commit: robot rightHand, 4 links, 3 joints
Links:
- added link indexSeg1; visual mesh filename=package://inmoov_urdf/meshes/rightHand/indexSeg1.stl scale=.001 .001 .001
- added link indexSeg2; visual mesh filename=package://inmoov_urdf/meshes/rightHand/indexSeg2.stl scale=.001 .001 .001
- added link indexSeg3; visual mesh filename=package://inmoov_urdf/meshes/rightHand/indexSeg3.stl scale=.001 .001 .001
- added link indexSeg4; visual mesh filename=package://inmoov_urdf/meshes/rightHand/indexSeg4.stl scale=.001 .001 .001
- added link indexSeg5; visual mesh filename=package://inmoov_urdf/meshes/rightHand/indexSeg5.stl scale=.001 .001 .001
Joints:
- added joint indexKnuck1.5: type fixed, parent indexSeg6, child indexSeg5
- added joint indexKnuck2: type revolute, parent indexSeg5, child indexSeg4, origin xyz=-0.0011 -0.0362 0.0007 rpy=0 0 0, limit lower=0.0 upper=-1.4 effort=1000.0 velocity=0.5
- added joint indexKnuck2.5: type fixed, parent indexSeg4, child indexSeg3
- added joint indexKnuck3: type revolute, parent indexSeg3, child indexSeg2, origin xyz=-0.00035 -0.02408 -0.00042 rpy=0 0 0, limit lower=0.0 upper=-0.87 effort=1000.0 velocity=0.5
- added joint indexKnuck3.5: type fixed, parent indexSeg2, child indexSeg1

Commit message: finished positioning the middle finger on the right hand

File: inmoov/inmoov_urdf/urdf/rightHand.urdf (robot description, URDF)
Before this commit: robot rightHand, 9 links, 8 joints
Links:
- added link middleSeg1; visual mesh filename=package://inmoov_urdf/meshes/rightHand/middleSeg1.stl scale=.001 .001 .001
- added link middleSeg2; visual mesh filename=package://inmoov_urdf/meshes/rightHand/middleSeg2.stl scale=.001 .001 .001
- added link middleSeg3; visual mesh filename=package://inmoov_urdf/meshes/rightHand/middleSeg3.stl scale=.001 .001 .001
- added link middleSeg4; visual mesh filename=package://inmoov_urdf/meshes/rightHand/middleSeg4.stl scale=.001 .001 .001
- added link middleSeg5; visual mesh filename=package://inmoov_urdf/meshes/rightHand/middleSeg5.stl scale=.001 .001 .001
- added link middleSeg6; visual mesh filename=package://inmoov_urdf/meshes/rightHand/middleSeg6.stl scale=.001 .001 .001
Joints:
- added joint middleKnuck1: type revolute, parent wristLarge, child middleSeg6, origin xyz=-0.0077 -0.0545 0.0107 rpy=0 0 0, limit lower=0.0 upper=-1.74533 effort=1000.0 velocity=0.5
- added joint middleKnuck1.5: type fixed, parent middleSeg6, child middleSeg5
- added joint middleKnuck2: type revolute, parent middleSeg5, child middleSeg4, origin xyz=-0.00235 -0.0388 0.00085 rpy=0 0 0, limit lower=0.0 upper=-1.4 effort=1000.0 velocity=0.5
- added joint middleKnuck2.5: type fixed, parent middleSeg4, child middleSeg3
- added joint middleKnuck3: type revolute, parent middleSeg3, child middleSeg2, origin xyz=-0.00035 -0.0259 -0.0005 rpy=0 0 0, limit lower=0.0 upper=-0.87 effort=1000.0 velocity=0.5
- added joint middleKnuck3.5: type fixed, parent middleSeg2, child middleSeg1

Commit message: finished positioning the ring finger

File: inmoov/inmoov_urdf/urdf/rightHand.urdf (robot description, URDF)
Before this commit: robot rightHand, 15 links, 14 joints
Links:
- added link ringSeg1; visual mesh filename=package://inmoov_urdf/meshes/rightHand/ringSeg1.stl scale=.001 .001 .001
- added link ringSeg2; visual mesh filename=package://inmoov_urdf/meshes/rightHand/ringSeg2.stl scale=.001 .001 .001
- added link ringSeg3; visual mesh filename=package://inmoov_urdf/meshes/rightHand/ringSeg3.stl scale=.001 .001 .001
- added link ringSeg4; visual mesh filename=package://inmoov_urdf/meshes/rightHand/ringSeg4.stl scale=.001 .001 .001
- added link ringSeg5; visual mesh filename=package://inmoov_urdf/meshes/rightHand/ringSeg5.stl scale=.001 .001 .001
- added link ringSeg6; visual mesh filename=package://inmoov_urdf/meshes/rightHand/ringSeg6.stl scale=.001 .001 .001
Joints:
- removed joint pinkyKnuck1
- added joint ringKnuck1.5: type fixed, parent ringSeg6, child ringSeg5
- added joint ringKnuck2: type revolute, parent ringSeg5, child ringSeg4, origin xyz=0.00007 -0.0346 0.00085 rpy=0 0 0, limit lower=0.0 upper=-1.4 effort=1000.0 velocity=0.5
- added joint ringKnuck2.5: type fixed, parent ringSeg4, child ringSeg3
- added joint ringKnuck3: type revolute, parent ringSeg3, child ringSeg2, origin xyz=-0.0003 -0.02295 -0.0005 rpy=0 0 0, limit lower=0.0 upper=-0.87 effort=1000.0 velocity=0.5
- added joint ringKnuck3.5: type fixed, parent ringSeg2, child ringSeg1
- added joint wristPinkyKnuck1: type revolute, parent wristLarge, child wristPinky, origin xyz=0.005 -0.0105 .0105 rpy=0 0 4.03171057, limit lower=0.0 upper=0.3 effort=1000.0 velocity=0.5
- added joint wristRingKnuck1: type revolute, parent wristLarge, child wristRing, origin xyz=0.005 -0.0105 0.0105 rpy=0 0 4.03171057, limit lower=0.0 upper=0.23 effort=1000.0 velocity=0.5
- joint ringKnuck1: child wristRing -> ringSeg6; limit lower=0.0 upper=0.23 effort=1000.0 velocity=0.5 -> lower=0.0 upper=-1.74533 effort=1000.0 velocity=0.5; origin xyz=0.005 -0.0105 0.0105 rpy=0 0 4.03171057 -> xyz=0.0164 0.035 0.0002 rpy=0 0 -3.945; parent wristLarge -> wristRing

Commit message: finished positioning the pinky finger

File: inmoov/inmoov_urdf/urdf/rightHand.urdf (robot description, URDF)
Before this commit: robot rightHand, 21 links, 20 joints
Links:
- added link pinkySeg1; visual mesh filename=package://inmoov_urdf/meshes/rightHand/pinkySeg1.stl scale=.001 .001 .001
- added link pinkySeg2; visual mesh filename=package://inmoov_urdf/meshes/rightHand/pinkySeg2.stl scale=.001 .001 .001
- added link pinkySeg3; visual mesh filename=package://inmoov_urdf/meshes/rightHand/pinkySeg3.stl scale=.001 .001 .001
- added link pinkySeg4; visual mesh filename=package://inmoov_urdf/meshes/rightHand/pinkySeg4.stl scale=.001 .001 .001
- added link pinkySeg5; visual mesh filename=package://inmoov_urdf/meshes/rightHand/pinkySeg5.stl scale=.001 .001 .001
- added link pinkySeg6; visual mesh filename=package://inmoov_urdf/meshes/rightHand/pinkySeg6.stl scale=.001 .001 .001
Joints:
- added joint pinkyKnuck1: type revolute, parent wristPinky, child pinkySeg6, origin xyz=-0.00765 0.04505 -0.0014 rpy=0 0 -3.785, limit lower=0.0 upper=-1.74533 effort=1000.0 velocity=0.5
- added joint pinkyKnuck1.5: type fixed, parent pinkySeg6, child pinkySeg5
- added joint pinkyKnuck2: type revolute, parent pinkySeg5, child pinkySeg4, origin xyz=0.00275 -0.0311 0.00085 rpy=0 0 0, limit lower=0.0 upper=-1.4 effort=1000.0 velocity=0.5
- added joint pinkyKnuck2.5: type fixed, parent pinkySeg4, child pinkySeg3
- added joint pinkyKnuck3: type revolute, parent pinkySeg3, child pinkySeg2, origin xyz=-0.0003 -0.02065 -0.0005 rpy=0 0 0, limit lower=0.0 upper=-0.87 effort=1000.0 velocity=0.5
- added joint pinkyKnuck3.5: type fixed, parent pinkySeg2, child pinkySeg1

Commit message: finished positioning the thumb, thumbSeg5.stl was a pain in the butt lol

File: inmoov/inmoov_urdf/urdf/rightHand.urdf (robot description, URDF)
Before this commit: robot rightHand, 27 links, 26 joints
Links:
- added link thumbSeg1; visual mesh filename=package://inmoov_urdf/meshes/rightHand/thumbSeg1.stl scale=.001 .001 .001
- added link thumbSeg2; visual mesh filename=package://inmoov_urdf/meshes/rightHand/thumbSeg2.stl scale=.001 .001 .001
- added link thumbSeg3; visual mesh filename=package://inmoov_urdf/meshes/rightHand/thumbSeg3.stl scale=.001 .001 .001
- added link thumbSeg4; visual mesh filename=package://inmoov_urdf/meshes/rightHand/thumbSeg4.stl scale=.001 .001 .001
- added link thumbSeg5; visual mesh filename=package://inmoov_urdf/meshes/rightHand/thumbSeg5.stl scale=.001 .001 .001
- added link wristThumb; visual mesh filename=package://inmoov_urdf/meshes/rightHand/wristThumb.stl scale=.001 .001 .001
Joints:
- added joint thumbKnuck0.5: type fixed, parent wristThumb, child thumbSeg5
- added joint thumbKnuck1: type revolute, parent thumbSeg5, child thumbSeg4, origin xyz=-0.025 0.02605 -0.00065 rpy=0 0.23 -2.423, limit lower=0.0 upper=-1.4 effort=1000.0 velocity=0.5
- added joint thumbKnuck1.5: type fixed, parent thumbSeg4, child thumbSeg3
- added joint thumbKnuck2: type revolute, parent thumbSeg3, child thumbSeg2, origin xyz=-0.00221 -0.035 0 rpy=0 0 0, limit lower=0.0 upper=-1.13 effort=1000.0 velocity=0.5
- added joint thumbKnuck2.5: type fixed, parent thumbSeg2, child thumbSeg1
- added joint wristThumbKnuck1: type revolute, parent wristLarge, child wristThumb, origin xyz=-0.0307 0.0206 0.0105 rpy=0 0 1.48, limit lower=0.0 upper=0.7 effort=1000.0 velocity=0.5
- joint wristPinkyKnuck1: origin xyz=0.005 -0.0105 .0105 rpy=0 0 4.03171057 -> xyz=0.005 -0.0105 0.0105 rpy=0 0 4.03171057

Commit message: finished collision model of the right Hand

File: inmoov/inmoov_urdf/urdf/rightHand.urdf (robot description, URDF)
Before this commit: robot rightHand, 33 links, 32 joints
Links:
- link indexSeg2: geometry collision cylinder length=0.025 radius=0.007; visual mesh filename=package://inmoov_urdf/meshes/rightHand/indexSeg2.stl scale=.001 .001 .001
- link indexSeg4: geometry collision cylinder length=0.02408 radius=0.008; visual mesh filename=package://inmoov_urdf/meshes/rightHand/indexSeg4.stl scale=.001 .001 .001
- link indexSeg6: geometry collision cylinder length=0.0362 radius=0.0085; visual mesh filename=package://inmoov_urdf/meshes/rightHand/indexSeg6.stl scale=.001 .001 .001
- link middleSeg2: geometry collision cylinder length=0.025 radius=0.007; visual mesh filename=package://inmoov_urdf/meshes/rightHand/middleSeg2.stl scale=.001 .001 .001
- link middleSeg4: geometry collision cylinder length=0.0259 radius=0.008; visual mesh filename=package://inmoov_urdf/meshes/rightHand/middleSeg4.stl scale=.001 .001 .001
- link middleSeg6: geometry collision cylinder length=0.0388 radius=0.009; visual mesh filename=package://inmoov_urdf/meshes/rightHand/middleSeg6.stl scale=.001 .001 .001
- link pinkySeg2: geometry collision cylinder length=0.02 radius=0.0057; visual mesh filename=package://inmoov_urdf/meshes/rightHand/pinkySeg2.stl scale=.001 .001 .001
- link pinkySeg4: geometry collision cylinder length=0.02065 radius=0.0067; visual mesh filename=package://inmoov_urdf/meshes/rightHand/pinkySeg4.stl scale=.001 .001 .001
- link pinkySeg6: geometry collision cylinder length=0.0311 radius=0.0073; visual mesh filename=package://inmoov_urdf/meshes/rightHand/pinkySeg6.stl scale=.001 .001 .001
- link ringSeg2: geometry collision cylinder length=0.023 radius=0.0065; visual mesh filename=package://inmoov_urdf/meshes/rightHand/ringSeg2.stl scale=.001 .001 .001
- link ringSeg4: geometry collision cylinder length=0.02295 radius=0.0075; visual mesh filename=package://inmoov_urdf/meshes/rightHand/ringSeg4.stl scale=.001 .001 .001
- link ringSeg6: geometry collision cylinder length=0.0346 radius=0.0085; visual mesh filename=package://inmoov_urdf/meshes/rightHand/ringSeg6.stl scale=.001 .001 .001
- link thumbSeg2: geometry collision cylinder length=0.024 radius=0.0083; visual mesh filename=package://inmoov_urdf/meshes/rightHand/thumbSeg2.stl scale=.001 .001 .001
- link thumbSeg4: geometry collision cylinder length=0.035 radius=0.0115; visual mesh filename=package://inmoov_urdf/meshes/rightHand/thumbSeg4.stl scale=.001 .001 .001
- link wristLarge: geometry collision box size=0.087 0.09 0.018; visual mesh filename=package://inmoov_urdf/meshes/rightHand/WristlargeV4.stl scale=.001 .001 .001
- link wristPinky: geometry collision box size=0.03 0.048 0.018; visual mesh filename=package://inmoov_urdf/meshes/rightHand/wristSmallPinky.stl scale=.001 .001 .001
- link wristRing: geometry collision box size=0.03 0.036 0.018; visual mesh filename=package://inmoov_urdf/meshes/rightHand/wristSmallRing.stl scale=.001 .001 .001
- link wristThumb: geometry collision box size=0.027 0.036 0.018; visual mesh filename=package://inmoov_urdf/meshes/rightHand/wristThumb.stl scale=.001 .001 .001
